Commit message: Change drc-hubo model feet to low-res version

File: data/models/drchubo-master/robots/drchubo.urdf (robot description, URDF)
Before this commit: robot drchubo, 40 links, 39 joints
Links:
- link Body_LAR: geometry collision mesh filename=package://drchubo/meshes/Body_LAR.stl; visual mesh filename=package://drchubo/meshes/Body_LAR.stl
- link Body_RAR: geometry collision mesh filename=package://drchubo/meshes/Body_RAR.stl; visual mesh filename=package://drchubo/meshes/Body_RAR.stl

Commit message: fix package path in drchubo urdf

File: data/models/drchubo-master/robots/drchubo.urdf (robot description, URDF)
Before this commit: robot drchubo, 40 links, 39 joints
Links:
- link Body_Hip: geometry collision mesh filename=package://vrc-golem/data/models/drchubo-master//meshes/Body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; visual mesh filename=package://vrc-golem/data/models/drchubo-master//meshes/Body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
- link Body_LAP: geometry collision mesh filename=package://vrc-golem/data/models/drchubo-master//meshes/Body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; visual mesh filename=package://vrc-golem/data/models/drchubo-master//meshes/Body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
- link Body_LAR: geometry collision mesh filename=package://vrc-golem/data/models/drchubo-master//meshes/Body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; visual mesh filename=package://vrc-golem/data/models/drchubo-master//meshes/Body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
- link Body_LEP: geometry collision mesh filename=package://vrc-golem/data/models/drchubo-master//meshes/Body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; visual mesh filename=package://vrc-golem/data/models/drchubo-master//meshes/Body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
- link Body_LF1: geometry collision mesh filename=package://vrc-golem/data/models/drchubo-master//meshes/Body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; visual mesh filename=package://vrc-golem/data/models/drchubo-master//meshes/Body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
- link Body_LF2: geometry collision mesh filename=package://vrc-golem/data/models/drchubo-master//meshes/Body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; visual mesh filename=package://vrc-golem/data/models/drchubo-master//meshes/Body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
- link Body_LF3: geometry collision mesh filename=package://vrc-golem/data/models/drchubo-master//meshes/Body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; visual mesh filename=package://vrc-golem/data/models/drchubo-master//meshes/Body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
- link Body_LHP: geometry collision mesh filename=package://vrc-golem/data/models/drchubo-master//meshes/Body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; visual mesh filename=package://vrc-golem/data/models/drchubo-master//meshes/Body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
- link Body_LHR: geometry collision mesh filename=package://vrc-golem/data/models/drchubo-master//meshes/Body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; visual mesh filename=package://vrc-golem/data/models/drchubo-master//meshes/Body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
- link Body_LHY: geometry collision mesh filename=package://vrc-golem/data/models/drchubo-master//meshes/Body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; visual mesh filename=package://vrc-golem/data/models/drchubo-master//meshes/Body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
- link Body_LKP: geometry collision mesh filename=package://vrc-golem/data/models/drchubo-master//meshes/Body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; visual mesh filename=package://vrc-golem/data/models/drchubo-master//meshes/Body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
- link Body_LSP: geometry collision mesh filename=package://vrc-golem/data/models/drchubo-master//meshes/Body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; visual mesh filename=package://vrc-golem/data/models/drchubo-master//meshes/Body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
- link Body_LSR: geometry collision mesh filename=package://vrc-golem/data/models/drchubo-master//meshes/Body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; visual mesh filename=package://vrc-golem/data/models/drchubo-master//meshes/Body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
- link Body_LSY: geometry collision mesh filename=package://vrc-golem/data/models/drchubo-master//meshes/Body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; visual mesh filename=package://vrc-golem/data/models/drchubo-master//meshes/Body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
- link Body_LWP: geometry collision mesh filename=package://vrc-golem/data/models/drchubo-master//meshes/Body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; visual mesh filename=package://vrc-golem/data/models/drchubo-master//meshes/Body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
- link Body_LWR: geometry collision mesh filename=package://vrc-golem/data/models/drchubo-master//meshes/Body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; visual mesh filename=package://vrc-golem/data/models/drchubo-master//meshes/Body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
- link Body_LWY: geometry collision mesh filename=package://vrc-golem/data/models/drchubo-master//meshes/Body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; visual mesh filename=package://vrc-golem/data/models/drchubo-master//meshes/Body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
- link Body_NKP: geometry collision mesh filename=package://vrc-golem/data/models/drchubo-master//meshes/Body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; visual mesh filename=package://vrc-golem/data/models/drchubo-master//meshes/Body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
- link Body_NKY: geometry collision mesh filename=package://vrc-golem/data/models/drchubo-master//meshes/Body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; visual mesh filename=package://vrc-golem/data/models/drchubo-master//meshes/Body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
- link Body_RAP: geometry collision mesh filename=package://vrc-golem/data/models/drchubo-master//meshes/Body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; visual mesh filename=package://vrc-golem/data/models/drchubo-master//meshes/Body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
- link Body_RAR: geometry collision mesh filename=package://vrc-golem/data/models/drchubo-master//meshes/Body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; visual mesh filename=package://vrc-golem/data/models/drchubo-master//meshes/Body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
- link Body_REP: geometry collision mesh filename=package://vrc-golem/data/models/drchubo-master//meshes/Body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; visual mesh filename=package://vrc-golem/data/models/drchubo-master//meshes/Body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
- link Body_RF1: geometry collision mesh filename=package://vrc-golem/data/models/drchubo-master//meshes/Body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; visual mesh filename=package://vrc-golem/data/models/drchubo-master//meshes/Body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
- link Body_RF2: geometry collision mesh filename=package://vrc-golem/data/models/drchubo-master//meshes/Body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; visual mesh filename=package://vrc-golem/data/models/drchubo-master//meshes/Body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
- link Body_RF3: geometry collision mesh filename=package://vrc-golem/data/models/drchubo-master//meshes/Body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; visual mesh filename=package://vrc-golem/data/models/drchubo-master//meshes/Body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
- link Body_RHP: geometry collision mesh filename=package://vrc-golem/data/models/drchubo-master//meshes/Body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; visual mesh filename=package://vrc-golem/data/models/drchubo-master//meshes/Body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
- link Body_RHR: geometry collision mesh filename=package://vrc-golem/data/models/drchubo-master//meshes/Body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; visual mesh filename=package://vrc-golem/data/models/drchubo-master//meshes/Body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
- link Body_RHY: geometry collision mesh filename=package://vrc-golem/data/models/drchubo-master//meshes/Body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; visual mesh filename=package://vrc-golem/data/models/drchubo-master//meshes/Body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
- link Body_RKP: geometry collision mesh filename=package://vrc-golem/data/models/drchubo-master//meshes/Body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; visual mesh filename=package://vrc-golem/data/models/drchubo-master//meshes/Body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
- link Body_RSP: geometry collision mesh filename=package://vrc-golem/data/models/drchubo-master//meshes/Body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; visual mesh filename=package://vrc-golem/data/models/drchubo-master//meshes/Body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
- link Body_RSR: geometry collision mesh filename=package://vrc-golem/data/models/drchubo-master//meshes/Body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; visual mesh filename=package://vrc-golem/data/models/drchubo-master//meshes/Body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
- link Body_RSY: geometry collision mesh filename=package://vrc-golem/data/models/drchubo-master//meshes/Body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; visual mesh filename=package://vrc-golem/data/models/drchubo-master//meshes/Body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
- link Body_RWP: geometry collision mesh filename=package://vrc-golem/data/models/drchubo-master//meshes/Body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; visual mesh filename=package://vrc-golem/data/models/drchubo-master//meshes/Body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
- link Body_RWR: geometry collision mesh filename=package://vrc-golem/data/models/drchubo-master//meshes/Body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; visual mesh filename=package://vrc-golem/data/models/drchubo-master//meshes/Body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
- link Body_RWY: geometry collision mesh filename=package://vrc-golem/data/models/drchubo-master//meshes/Body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; visual mesh filename=package://vrc-golem/data/models/drchubo-master//meshes/Body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
- link Body_Torso: geometry collision mesh filename=package://vrc-golem/data/models/drchubo-master//meshes/Body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; visual mesh filename=package://vrc-golem/data/models/drchubo-master//meshes/Body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

Commit message: fixed package path in drchubo.urdf

File: data/models/drchubo-master/robots/drchubo.urdf (robot description, URDF)
Before this commit: robot drchubo, 40 links, 39 joints
Links:
- link Body_Hip: geometry collision mesh filename=package://drchubo/data/models/drchubo-master//meshes/Body_H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; visual mesh filename=package://drchubo/data/models/drchubo-master//meshes/Body_H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
- link Body_LAP: geometry collision mesh filename=package://drchubo/data/models/drchubo-master//meshes/Body_L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; visual mesh filename=package://drchubo/data/models/drchubo-master//meshes/Body_L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
- link Body_LAR: geometry collision mesh filename=package://drchubo/data/models/drchubo-master//meshes/Body_L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; visual mesh filename=package://drchubo/data/models/drchubo-master//meshes/Body_L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
- link Body_LEP: geometry collision mesh filename=package://drchubo/data/models/drchubo-master//meshes/Body_L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; visual mesh filename=package://drchubo/data/models/drchubo-master//meshes/Body_L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
- link Body_LF1: geometry collision mesh filename=package://drchubo/data/models/drchubo-master//meshes/Body_L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; visual mesh filename=package://drchubo/data/models/drchubo-master//meshes/Body_L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
- link Body_LF2: geometry collision mesh filename=package://drchubo/data/models/drchubo-master//meshes/Body_L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; visual mesh filename=package://drchubo/data/models/drchubo-master//meshes/Body_L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
- link Body_LF3: geometry collision mesh filename=package://drchubo/data/models/drchubo-master//meshes/Body_L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; visual mesh filename=package://drchubo/data/models/drchubo-master//meshes/Body_L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
- link Body_LHP: geometry collision mesh filename=package://drchubo/data/models/drchubo-master//meshes/Body_L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; visual mesh filename=package://drchubo/data/models/drchubo-master//meshes/Body_L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
- link Body_LHR: geometry collision mesh filename=package://drchubo/data/models/drchubo-master//meshes/Body_L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; visual mesh filename=package://drchubo/data/models/drchubo-master//meshes/Body_L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
- link Body_LHY: geometry collision mesh filename=package://drchubo/data/models/drchubo-master//meshes/Body_L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; visual mesh filename=package://drchubo/data/models/drchubo-master//meshes/Body_L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
- link Body_LKP: geometry collision mesh filename=package://drchubo/data/models/drchubo-master//meshes/Body_L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; visual mesh filename=package://drchubo/data/models/drchubo-master//meshes/Body_L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
- link Body_LSP: geometry collision mesh filename=package://drchubo/data/models/drchubo-master//meshes/Body_L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; visual mesh filename=package://drchubo/data/models/drchubo-master//meshes/Body_L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
- link Body_LSR: geometry collision mesh filename=package://drchubo/data/models/drchubo-master//meshes/Body_L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; visual mesh filename=package://drchubo/data/models/drchubo-master//meshes/Body_L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
- link Body_LSY: geometry collision mesh filename=package://drchubo/data/models/drchubo-master//meshes/Body_L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; visual mesh filename=package://drchubo/data/models/drchubo-master//meshes/Body_L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
- link Body_LWP: geometry collision mesh filename=package://drchubo/data/models/drchubo-master//meshes/Body_L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; visual mesh filename=package://drchubo/data/models/drchubo-master//meshes/Body_L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
- link Body_LWR: geometry collision mesh filename=package://drchubo/data/models/drchubo-master//meshes/Body_L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; visual mesh filename=package://drchubo/data/models/drchubo-master//meshes/Body_L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
- link Body_LWY: geometry collision mesh filename=package://drchubo/data/models/drchubo-master//meshes/Body_L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; visual mesh filename=package://drchubo/data/models/drchubo-master//meshes/Body_L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
- link Body_NKP: geometry collision mesh filename=package://drchubo/data/models/drchubo-master//meshes/Body_N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; visual mesh filename=package://drchubo/data/models/drchubo-master//meshes/Body_N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
- link Body_NKY: geometry collision mesh filename=package://drchubo/data/models/drchubo-master//meshes/Body_N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; visual mesh filename=package://drchubo/data/models/drchubo-master//meshes/Body_N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
- link Body_RAP: geometry collision mesh filename=package://drchubo/data/models/drchubo-master//meshes/Body_R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; visual mesh filename=package://drchubo/data/models/drchubo-master//meshes/Body_R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
- link Body_RAR: geometry collision mesh filename=package://drchubo/data/models/drchubo-master//meshes/Body_R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; visual mesh filename=package://drchubo/data/models/drchubo-master//meshes/Body_R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
- link Body_REP: geometry collision mesh filename=package://drchubo/data/models/drchubo-master//meshes/Body_R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; visual mesh filename=package://drchubo/data/models/drchubo-master//meshes/Body_R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
- link Body_RF1: geometry collision mesh filename=package://drchubo/data/models/drchubo-master//meshes/Body_R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; visual mesh filename=package://drchubo/data/models/drchubo-master//meshes/Body_R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
- link Body_RF2: geometry collision mesh filename=package://drchubo/data/models/drchubo-master//meshes/Body_R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; visual mesh filename=package://drchubo/data/models/drchubo-master//meshes/Body_R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
- link Body_RF3: geometry collision mesh filename=package://drchubo/data/models/drchubo-master//meshes/Body_R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; visual mesh filename=package://drchubo/data/models/drchubo-master//meshes/Body_R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
- link Body_RHP: geometry collision mesh filename=package://drchubo/data/models/drchubo-master//meshes/Body_R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; visual mesh filename=package://drchubo/data/models/drchubo-master//meshes/Body_R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
- link Body_RHR: geometry collision mesh filename=package://drchubo/data/models/drchubo-master//meshes/Body_R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; visual mesh filename=package://drchubo/data/models/drchubo-master//meshes/Body_R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
- link Body_RHY: geometry collision mesh filename=package://drchubo/data/models/drchubo-master//meshes/Body_R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; visual mesh filename=package://drchubo/data/models/drchubo-master//meshes/Body_R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
- link Body_RKP: geometry collision mesh filename=package://drchubo/data/models/drchubo-master//meshes/Body_R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; visual mesh filename=package://drchubo/data/models/drchubo-master//meshes/Body_R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
- link Body_RSP: geometry collision mesh filename=package://drchubo/data/models/drchubo-master//meshes/Body_R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; visual mesh filename=package://drchubo/data/models/drchubo-master//meshes/Body_R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
- link Body_RSR: geometry collision mesh filename=package://drchubo/data/models/drchubo-master//meshes/Body_R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; visual mesh filename=package://drchubo/data/models/drchubo-master//meshes/Body_R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
- link Body_RSY: geometry collision mesh filename=package://drchubo/data/models/drchubo-master//meshes/Body_R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; visual mesh filename=package://drchubo/data/models/drchubo-master//meshes/Body_R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
- link Body_RWP: geometry collision mesh filename=package://drchubo/data/models/drchubo-master//meshes/Body_R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; visual mesh filename=package://drchubo/data/models/drchubo-master//meshes/Body_R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
- link Body_RWR: geometry collision mesh filename=package://drchubo/data/models/drchubo-master//meshes/Body_R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; visual mesh filename=package://drchubo/data/models/drchubo-master//meshes/Body_R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
- link Body_RWY: geometry collision mesh filename=package://drchubo/data/models/drchubo-master//meshes/Body_R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; visual mesh filename=package://drchubo/data/models/drchubo-master//meshes/Body_R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
- link Body_Torso: geometry collision mesh filename=package://drchubo/data/models/drchubo-master//meshes/Body_T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; visual mesh filename=package://drchubo/data/models/drchubo-master//meshes/Body_T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

Commit message: Erased an extra backslash / from mesh filenames in drchubo.urdf

File: data/models/drchubo-master/robots/drchubo.urdf (robot description, URDF)
Before this commit: robot drchubo, 40 links, 39 joints
Links:
- link Body_Hip: geometry collision mesh filename=package://drchubo/data/models/drchubo-master/meshes/Body_Hi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; visual mesh filename=package://drchubo/data/models/drchubo-master/meshes/Body_Hi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
- link Body_LAP: geometry collision mesh filename=package://drchubo/data/models/drchubo-master/meshes/Body_LA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; visual mesh filename=package://drchubo/data/models/drchubo-master/meshes/Body_LA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
- link Body_LAR: geometry collision mesh filename=package://drchubo/data/models/drchubo-master/meshes/Body_LA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; visual mesh filename=package://drchubo/data/models/drchubo-master/meshes/Body_LA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
- link Body_LEP: geometry collision mesh filename=package://drchubo/data/models/drchubo-master/meshes/Body_LE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; visual mesh filename=package://drchubo/data/models/drchubo-master/meshes/Body_LE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
- link Body_LF1: geometry collision mesh filename=package://drchubo/data/models/drchubo-master/meshes/Body_LF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; visual mesh filename=package://drchubo/data/models/drchubo-master/meshes/Body_LF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
- link Body_LF2: geometry collision mesh filename=package://drchubo/data/models/drchubo-master/meshes/Body_LF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; visual mesh filename=package://drchubo/data/models/drchubo-master/meshes/Body_LF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
- link Body_LF3: geometry collision mesh filename=package://drchubo/data/models/drchubo-master/meshes/Body_LF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; visual mesh filename=package://drchubo/data/models/drchubo-master/meshes/Body_LF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
- link Body_LHP: geometry collision mesh filename=package://drchubo/data/models/drchubo-master/meshes/Body_LH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; visual mesh filename=package://drchubo/data/models/drchubo-master/meshes/Body_LH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
- link Body_LHR: geometry collision mesh filename=package://drchubo/data/models/drchubo-master/meshes/Body_LH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; visual mesh filename=package://drchubo/data/models/drchubo-master/meshes/Body_LH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
- link Body_LHY: geometry collision mesh filename=package://drchubo/data/models/drchubo-master/meshes/Body_LH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; visual mesh filename=package://drchubo/data/models/drchubo-master/meshes/Body_LH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
- link Body_LKP: geometry collision mesh filename=package://drchubo/data/models/drchubo-master/meshes/Body_LK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; visual mesh filename=package://drchubo/data/models/drchubo-master/meshes/Body_LK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
- link Body_LSP: geometry collision mesh filename=package://drchubo/data/models/drchubo-master/meshes/Body_LS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; visual mesh filename=package://drchubo/data/models/drchubo-master/meshes/Body_LS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
- link Body_LSR: geometry collision mesh filename=package://drchubo/data/models/drchubo-master/meshes/Body_LS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; visual mesh filename=package://drchubo/data/models/drchubo-master/meshes/Body_LS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
- link Body_LSY: geometry collision mesh filename=package://drchubo/data/models/drchubo-master/meshes/Body_LS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; visual mesh filename=package://drchubo/data/models/drchubo-master/meshes/Body_LS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
- link Body_LWP: geometry collision mesh filename=package://drchubo/data/models/drchubo-master/meshes/Body_LW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; visual mesh filename=package://drchubo/data/models/drchubo-master/meshes/Body_LW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
- link Body_LWR: geometry collision mesh filename=package://drchubo/data/models/drchubo-master/meshes/Body_LW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; visual mesh filename=package://drchubo/data/models/drchubo-master/meshes/Body_LW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
- link Body_LWY: geometry collision mesh filename=package://drchubo/data/models/drchubo-master/meshes/Body_LW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; visual mesh filename=package://drchubo/data/models/drchubo-master/meshes/Body_LW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
- link Body_NKP: geometry collision mesh filename=package://drchubo/data/models/drchubo-master/meshes/Body_NK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; visual mesh filename=package://drchubo/data/models/drchubo-master/meshes/Body_NK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
- link Body_NKY: geometry collision mesh filename=package://drchubo/data/models/drchubo-master/meshes/Body_NK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; visual mesh filename=package://drchubo/data/models/drchubo-master/meshes/Body_NK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
- link Body_RAP: geometry collision mesh filename=package://drchubo/data/models/drchubo-master/meshes/Body_RA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; visual mesh filename=package://drchubo/data/models/drchubo-master/meshes/Body_RA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
- link Body_RAR: geometry collision mesh filename=package://drchubo/data/models/drchubo-master/meshes/Body_RA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; visual mesh filename=package://drchubo/data/models/drchubo-master/meshes/Body_RA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
- link Body_REP: geometry collision mesh filename=package://drchubo/data/models/drchubo-master/meshes/Body_RE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; visual mesh filename=package://drchubo/data/models/drchubo-master/meshes/Body_RE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
- link Body_RF1: geometry collision mesh filename=package://drchubo/data/models/drchubo-master/meshes/Body_RF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; visual mesh filename=package://drchubo/data/models/drchubo-master/meshes/Body_RF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
- link Body_RF2: geometry collision mesh filename=package://drchubo/data/models/drchubo-master/meshes/Body_RF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; visual mesh filename=package://drchubo/data/models/drchubo-master/meshes/Body_RF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
- link Body_RF3: geometry collision mesh filename=package://drchubo/data/models/drchubo-master/meshes/Body_RF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; visual mesh filename=package://drchubo/data/models/drchubo-master/meshes/Body_RF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
- link Body_RHP: geometry collision mesh filename=package://drchubo/data/models/drchubo-master/meshes/Body_RH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; visual mesh filename=package://drchubo/data/models/drchubo-master/meshes/Body_RH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
- link Body_RHR: geometry collision mesh filename=package://drchubo/data/models/drchubo-master/meshes/Body_RH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; visual mesh filename=package://drchubo/data/models/drchubo-master/meshes/Body_RH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
- link Body_RHY: geometry collision mesh filename=package://drchubo/data/models/drchubo-master/meshes/Body_RH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; visual mesh filename=package://drchubo/data/models/drchubo-master/meshes/Body_RH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
- link Body_RKP: geometry collision mesh filename=package://drchubo/data/models/drchubo-master/meshes/Body_RK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; visual mesh filename=package://drchubo/data/models/drchubo-master/meshes/Body_RK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
- link Body_RSP: geometry collision mesh filename=package://drchubo/data/models/drchubo-master/meshes/Body_RS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; visual mesh filename=package://drchubo/data/models/drchubo-master/meshes/Body_RS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
- link Body_RSR: geometry collision mesh filename=package://drchubo/data/models/drchubo-master/meshes/Body_RS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; visual mesh filename=package://drchubo/data/models/drchubo-master/meshes/Body_RS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
- link Body_RSY: geometry collision mesh filename=package://drchubo/data/models/drchubo-master/meshes/Body_RS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; visual mesh filename=package://drchubo/data/models/drchubo-master/meshes/Body_RS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
- link Body_RWP: geometry collision mesh filename=package://drchubo/data/models/drchubo-master/meshes/Body_RW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; visual mesh filename=package://drchubo/data/models/drchubo-master/meshes/Body_RW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
- link Body_RWR: geometry collision mesh filename=package://drchubo/data/models/drchubo-master/meshes/Body_RW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; visual mesh filename=package://drchubo/data/models/drchubo-master/meshes/Body_RW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
- link Body_RWY: geometry collision mesh filename=package://drchubo/data/models/drchubo-master/meshes/Body_RW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; visual mesh filename=package://drchubo/data/models/drchubo-master/meshes/Body_RW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
- link Body_Torso: geometry collision mesh filename=package://drchubo/data/models/drchubo-master/meshes/Body_To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; visual mesh filename=package://drchubo/data/models/drchubo-master/meshes/Body_To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
