Commit message: hubo-urdf: fix joint limits on LF3 and RF3

File: data/models/drchubo-master/robots/drchubo.golem.urdf (robot description, URDF)
Before this commit: robot drchubo, 40 links, 39 joints
Joints:
- joint LF3: limit lower=-1.1 upper=.1 effort=100.0 velocity=10.0 -> lower=-0.1 upper=1.1 effort=100.0 velocity=10.0
- joint RF3: limit lower=-1.1 upper=.1 effort=100.0 velocity=10.0 -> lower=-0.1 upper=1.1 effort=100.0 velocity=10.0
