Commit message: models: drcsim-2.6 atlas

File: data/models/atlas/atlas-vrcgolem.urdf (robot description, URDF)
Before this commit: robot atlas, 41 links, 40 joints
Links:
- link head: geometry collision box size=0.0468 0.12 0.1184; collision box size=0.1311 0.12 0.0591
- link hokuyo_link: geometry collision box size=0.08 0.06 0.04238; collision cylinder length=0.047 radius=0.024425
- link l_clav: geometry collision box size=0.13 0.15 0.05; collision cylinder length=0.1525 radius=0.045
- link l_farm: geometry collision box size=0.135 0.1 0.045; collision cylinder length=0.125 radius=0.045
- link l_foot: geometry collision box size=0.26 0.124887 0.05; visual mesh filename=meshes/l_foot.dae scale=1 1 1
- link l_hand: geometry collision box size=0.13 0.09 0.07; collision cylinder length=0.05 radius=0.03
- link l_larm: geometry collision box size=0.135 0.15 0.06; collision cylinder length=0.125 radius=0.045
- link l_lglut: geometry collision cylinder length=0.060306 radius=0.02009687; collision cylinder length=0.12 radius=0.02
- link l_lleg: geometry collision cylinder length=0.40 radius=0.07; visual mesh filename=meshes/l_lleg.dae scale=1.0 1.0 1.0
- link l_scap: geometry collision box size=0.15 0.15 0.06; collision cylinder length=0.125 radius=0.045
- link l_talus: geometry collision cylinder length=0.010059 radius=0.010348; collision cylinder length=0.029542 radius=0.010181
- link l_uarm: geometry collision box size=0.04 0.07 0.13; collision cylinder length=0.125 radius=0.045
- link l_uglut: geometry collision cylinder length=0.078396 radius=0.019096; collision cylinder length=0.080842 radius=0.019841
- link l_uleg: geometry collision cylinder length=0.10 radius=0.1; collision cylinder length=0.15 radius=0.07
- link ltorso: geometry visual mesh filename=meshes/ltorso.dae scale=1 1 1
- link mtorso: geometry collision cylinder length=0.02 radius=0.015; collision cylinder length=0.02 radius=0.015
- link pelvis: geometry collision box size=0.1 0.15 0.2; collision cylinder length=0.05 radius=0.16
- link r_clav: geometry collision box size=0.13 0.15 0.05; collision cylinder length=0.1525 radius=0.045
- link r_farm: geometry collision box size=0.135 0.1 0.045; collision cylinder length=0.125 radius=0.045
- link r_foot: geometry collision box size=0.26 0.124887 0.05; visual mesh filename=meshes/r_foot.dae scale=1 1 1
- link r_hand: geometry collision box size=0.13 0.09 0.07; collision cylinder length=0.05 radius=0.03
- link r_larm: geometry collision box size=0.135 0.15 0.06; collision cylinder length=0.125 radius=0.045
- link r_lglut: geometry collision cylinder length=0.060306 radius=0.02009687; collision cylinder length=0.12 radius=0.02
- link r_lleg: geometry collision cylinder length=0.40 radius=0.07; visual mesh filename=meshes/r_lleg.dae scale=1.0 1.0 1.0
- link r_scap: geometry collision box size=0.15 0.15 0.06; collision cylinder length=0.125 radius=0.045
- link r_talus: geometry collision cylinder length=0.010059 radius=0.010348; collision cylinder length=0.029542 radius=0.010181
- link r_uarm: geometry collision box size=0.04 0.07 0.13; collision cylinder length=0.125 radius=0.045
- link r_uglut: geometry collision cylinder length=0.078396 radius=0.019096; collision cylinder length=0.080842 radius=0.019841
- link r_uleg: geometry collision cylinder length=0.10 radius=0.1; collision cylinder length=0.15 radius=0.07
- link utorso: geometry collision box size=0.3188 0.24 0.3162; collision cylinder length=0.22375 radius=0.0363

File: data/models/atlas/multisense_sl_description/multisense_sl_description.urdf (robot description, URDF)
Before this commit: robot atlas, 11 links, 10 joints
Links:
- added link head_imu_link, mass 1e-5; visual box size=0.01 0.01 0.01
- link center_bottom_led_frame: mass 0.1 -> 1e-5
- link center_top_led_frame: mass 0.1 -> 1e-5
- link head: mass 1.4199 -> 1.41984; geometry collision box size=0.0468 0.12 0.1184; collision box size=0.1311 0.12 0.0591
- link head_hokuyo_frame: mass 0.01 -> 1e-5
- link hokuyo_link: mass 0.057664 -> 0.057654; geometry collision box size=0.08 0.06 0.04238; collision cylinder length=0.047 radius=0.024425
- link left_camera_frame: mass 0.1 -> 1e-5
- link left_led_frame: mass 0.1 -> 1e-5
- link right_camera_frame: mass 0.1 -> 1e-5
- link right_led_frame: mass 0.1 -> 1e-5
Joints:
- added joint head_imu_joint: type fixed, parent head, child head_imu_link, origin xyz=-0.0475 0.035 0.0 rpy=0 0 0

Commit message: models: lowered right leg lhy to match left leg limits
Because: symmetry.

File: data/models/atlas/atlas-vrcgolem.urdf (robot description, URDF)
Before this commit: robot atlas, 41 links, 40 joints
Joints:
- joint l_leg_lhy: limit lower=-1.75 upper=0.524 effort=260 velocity=12 -> lower=-1.745 upper=0.524 effort=260 velocity=12

File: data/models/atlas/atlas.urdf (robot description, URDF)
Before this commit: robot atlas, 41 links, 40 joints
Joints:
- joint l_leg_lhy: limit lower=-1.75 upper=0.524 effort=260 velocity=12 -> lower=-1.745 upper=0.524 effort=260 velocity=12
